File: home_pwm.kicad_pcb (KiCad board)
At the start: 2 copper layers, 75 x 75 mm, 39 parts, among them J1 X977B06, J2 IDC-06, Q1 IRLR3410, Q2 IRLR3410, Q3 L-7113P3C, U1 ATmega8A-16AU, U2 L7805CDT, U3 IR25600, Y1 16 MHz

Commit message: PCB traced
Parts:
- added C13: 220n, NevaDA:C_0603, B.Cu at (79.5, 95.0)
- added C14: 220n, NevaDA:C_0603, B.Cu at (113.5, 82.0)
- added C15: 220n, NevaDA:C_0603, B.Cu at (115.5, 82.0)
- added D2: TO-5050BC, NevaDA:LED_RGB_5050-6, F.Cu at (88.0, 107.0)
- added R14: 22, NevaDA:R_1206, B.Cu at (103.0, 113.5)
- added R15: 22, NevaDA:R_1206, B.Cu at (116.0, 113.5)
- added R16: 1k, NevaDA:R_0603, B.Cu at (86.9, 91.8)
- added R17: 1k, NevaDA:R_0603, B.Cu at (86.9, 89.4)
- added R18: 1k, NevaDA:R_0603, B.Cu at (86.9, 86.9)
- added R19: 10k, NevaDA:R_0603, B.Cu at (109.5, 82.0)
- added R20: 10k, NevaDA:R_0603, B.Cu at (111.5, 82.0)
- added SW1: SW, NevaDA:SW_PUSH_6mm, F.Cu at (119.5, 88.5)
- added SW2: SW, NevaDA:SW_PUSH_6mm, F.Cu at (119.5, 97.5)
- added TP5: TestPoint, NevaDA:1Pin, F.Cu at (77.5, 85.0)
- TP1, TP3: footprint NevaDA:Screw_M3_9mm -> NevaDA:Screw_M3_6mm
- moved C5 17.5 mm to (107.5, 90.0)
- moved R4 9.62 mm to (76.5, 129.5), turned to 0 degrees
- moved D1 7.78 mm to (88.5, 133.0)
- moved Q1 4.50 mm to (105.0, 124.5)
- moved R5 4.00 mm to (68.0, 130.0)
- moved R1 3.50 mm to (76.5, 135.0)
- moved R6 3.50 mm to (68.0, 121.5)
- moved R10 2.92 mm to (106.0, 113.5), turned to 90 degrees
- moved C7 2.00 mm to (68.0, 110.0)
- moved R7 1.00 mm to (104.0, 99.0)
- moved R8 1.00 mm to (104.0, 97.0)
- moved C12 0.50 mm to (93.5, 84.0)
- moved C9 0.50 mm to (114.5, 105.0)
- moved R12 0.50 mm to (87.5, 84.0)
- moved R13 0.50 mm to (90.5, 83.0)
Connections:
- U1 pad 1: Net-(U1-Pad1) -> /BTN1
- U1 pad 2: Net-(U1-Pad2) -> /BTN2
- U1 pad 23: Net-(U1-Pad23) -> /LED_1
- U1 pad 24: Net-(U1-Pad24) -> /LED_2
- U1 pad 25: /OPTIC -> /LED_3
- U1 pad 26: Net-(U1-Pad26) -> /OPTIC
Routing:
- net GNDD: track 0.00 -> 513.8 mm, vias 0 -> 96
- net +5V: track 0.00 -> 120.7 mm, vias 0 -> 3
- net /SWITCH_CMOS: track 0.00 -> 74.1 mm, vias 0 -> 2
- net /RST: track 0.00 -> 49.9 mm, vias 0 -> 2
- net +12V: track 0.00 -> 40.9 mm
- net /BTN2: track 0.00 -> 37.0 mm
- net /SCK: track 0.00 -> 34.6 mm, vias 0 -> 1
- net /MISO: track 0.00 -> 30.3 mm, vias 0 -> 1
- net /BTN1: track 0.00 -> 30.2 mm
- net /MOSI: track 0.00 -> 25.9 mm, vias 0 -> 1
- net Net-(C10-Pad1): track 0.00 -> 22.5 mm
- net Net-(D2-Pad6): track 0.00 -> 18.9 mm, vias 0 -> 1
- net Net-(D2-Pad4): track 0.00 -> 16.6 mm, vias 0 -> 1
- net Net-(R11-Pad2): track 0.00 -> 15.8 mm
- net /XTAL2: track 0.00 -> 15.7 mm
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- added copper zone on B.Cu, net /OUT1
- added copper zone on B.Cu, net /OUT2
Other:
- outline, holes or cut-outs redrawn
- net class Default: clearance 0.2 -> 0.3; trace_width 0.25 -> 0.3
- rule trace_clearance: 0.2 -> 0.3
- rule trace_min: 0.2 -> 0.3
- board text added: "+"
- board text added: "+12V"
- board text added: "+5V"
- board text added: "-"
- board text added: "GND"
- board text added: "Made in Russia"
- board text added: "OUT A"
- board text added: "OUT B"
- board text added: "OUTPUT"
- board text added: "PWR"
- board text added: "SW"
- board text added: "SWITCH"
- board text added: "Sensor"
- board text added: "Status LED: R - OFF G - Level 1 C - Level 2 B - Level 3 Y - Auto"

Commit message: Gerbers
Routing:
- net Net-(Q2-Pad1): track 13.8 -> 12.4 mm
Other:
- board text added: "ADJUST"
Changed lines of the file:
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@@
   (general
     (thickness 1.6)
-    (drawings 40)
-    (tracks 564)
+    (drawings 41)
+    (tracks 567)
     (zones 0)
     (modules 53)
@@
   )
   (setup
-    (last_trace_width 0.3)
+    (last_trace_width 0.6)
     (user_trace_width 0.3)
     (user_trace_width 0.4)
@@
       (layerselection 0x010fc_ffffffff)
       (usegerberextensions false)
-      (usegerberattributes false)
+      (usegerberattributes true)
       (usegerberadvancedattributes false)
-      (creategerberjobfile false)
+      (creategerberjobfile true)
       (excludeedgelayer true)
       (linewidth 0.100000)
@@
       (outputformat 1)
       (mirror false)
-      (drillshape 1)
+      (drillshape 0)
       (scaleselection 1)
       (outputdirectory ""))
@@
     (tags "resistor 1206")
     (attr smd)
-    (fp_text reference R10 (at 0 2.5 90) (layer B.SilkS)
+    (fp_text reference R10 (at 1 2.5 90) (layer B.SilkS)
       (effects (font (size 1 1) (thickness 0.15)) (justify mirror))
     )
@@
     (descr "10 pins through hole IDC header")
     (tags "IDC header socket VASCH")
-    (fp_text reference J2 (at 8 -1.5) (layer F.SilkS)
+    (fp_text reference J2 (at 8 -1) (layer F.SilkS)
       (effects (font (size 1 1) (thickness 0.15)))
     )
@@
       (rotate (xyz 0 0 0))
     )
+  )
+  (gr_text ADJUST (at 116 95.5 90) (layer F.SilkS)
+    (effects (font (size 2.5 2.5) (thickness 0.3)))
   )
   (gr_text "Made in Russia" (at 100 146) (layer B.SilkS)
@@
   (segment (start 104.6 84) (end 105 83.6) (width 0.3) (layer B.Cu) (net 2))
   (segment (start 103 84) (end 104.6 84) (width 0.3) (layer B.Cu) (net 2))
-  (segment (start 76.5 128.5) (end 77.5 127.5) (width 0.3) (layer B.Cu) (net 2))
-  (via (at 77.5 127.5) (size 0.8) (drill 0.4) (layers F.Cu B.Cu) (net 2))
   (via (at 98 87.5) (size 0.8) (drill 0.4) (layers F.Cu B.Cu) (net 2))
-  (segment (start 92.5 92.5) (end 97.5 87.5) (width 0.3) (layer F.Cu) (net 2))
-  (segment (start 92.5 105.5) (end 92.5 92.5) (width 0.3) (layer F.Cu) (net 2))
-  (segment (start 77.5 109.5) (end 80 107) (width 0.3) (layer F.Cu) (net 2))
-  (segment (start 77.5 127.5) (end 77.5 109.5) (width 0.3) (layer F.Cu) (net 2))
-  (segment (start 80 107) (end 91 107) (width 0.3) (layer F.Cu) (net 2))
-  (segment (start 97.5 87.5) (end 98 87.5) (width 0.3) (layer F.Cu) (net 2))
-  (segment (start 91 107) (end 92.5 105.5) (width 0.3) (layer F.Cu) (net 2))
-  (segment (start 76.5 134.1) (end 76.5 128.5) (width 0.3) (layer B.Cu) (net 2))
   (segment (start 102.8 86.7) (end 102.8 85.65) (width 0.3) (layer B.Cu) (net 2))
   (segment (start 98.5 87) (end 102.5 87) (width 0.3) (layer B.Cu) (net 2))
   (segment (start 102.5 87) (end 102.8 86.7) (width 0.3) (layer B.Cu) (net 2))
   (segment (start 98 87.5) (end 98.5 87) (width 0.3) (layer B.Cu) (net 2))
+  (segment (start 77.5 109.5) (end 77.5 127.5) (width 0.3) (layer F.Cu) (net 2))
+  (segment (start 98 87.5) (end 92.5 93) (width 0.3) (layer F.Cu) (net 2))
+  (segment (start 92.5 93) (end 92.5 105.5) (width 0.3) (layer F.Cu) (net 2))
+  (segment (start 92.5 105.5) (end 91 107) (width 0.3) (layer F.Cu) (net 2))
+  (segment (start 91 107) (end 80 107) (width 0.3) (layer F.Cu) (net 2))
+  (segment (start 80 107) (end 77.5 109.5) (width 0.3) (layer F.Cu) (net 2))
+  (via (at 77 132.5) (size 0.8) (drill 0.4) (layers F.Cu B.Cu) (net 2))
+  (segment (start 76.5 134.1) (end 76.5 133) (width 0.3) (layer B.Cu) (net 2))
+  (segment (start 76.5 133) (end 77 132.5) (width 0.3) (layer B.Cu) (net 2))
+  (segment (start 77.5 132) (end 77.5 127.5) (width 0.3) (layer F.Cu) (net 2))
+  (segment (start 77 132.5) (end 77.5 132) (width 0.3) (layer F.Cu) (net 2))
   (segment (start 95.65 92) (end 99.5 92) (width 0.4) (layer B.Cu) (net 3) (status 10))
   (segment (start 101.9 89.6) (end 104.35 89.6) (width 0.4) (layer B.Cu) (net 3) (status 20))
@@
   (segment (start 103 117) (end 103.5 117.5) (width 0.8) (layer B.Cu) (net 16))
   (segment (start 103 115.1) (end 103 117) (width 0.8) (layer B.Cu) (net 16))
-  (segment (start 117.6 110) (end 121.5 110) (width 0.6) (layer B.Cu) (net 17))
-  (segment (start 122.3 110.8) (end 125.22 110.8) (width 0.6) (layer B.Cu) (net 17))
-  (segment (start 121.5 110) (end 122.3 110.8) (width 0.6) (layer B.Cu) (net 17))
-  (segment (start 119.6 113.5) (end 122.3 110.8) (width 0.6) (layer B.Cu) (net 17))
-  (segment (start 117.6 113.5) (end 119.6 113.5) (width 0.6) (layer B.Cu) (net 17))
+  (segment (start 118.8 110) (end 119.5 110.7) (width 0.6) (layer B.Cu) (net 17))
+  (segment (start 117.6 110) (end 118.8 110) (width 0.6) (layer B.Cu) (net 17))
+  (segment (start 119.5 113) (end 119 113.5) (width 0.6) (layer B.Cu) (net 17))
+  (segment (start 119.5 110.7) (end 119.5 113) (width 0.6) (layer B.Cu) (net 17))
+  (segment (start 117.6 113.5) (end 119 113.5) (width 0.6) (layer B.Cu) (net 17))
+  (segment (start 119.6 110.8) (end 119.5 110.7) (width 0.6) (layer B.Cu) (net 17))
+  (segment (start 125.22 110.8) (end 119.6 110.8) (width 0.6) (layer B.Cu) (net 17))
   (segment (start 87.6 83) (end 87.5 83.1) (width 0.3) (layer B.Cu) (net 18))
   (segment (start 89.6 83) (end 87.6 83) (width 0.3) (layer B.Cu) (net 18))
