File: home_pwm.sch (KiCad schematic (older format))
At the start: 11 parts

Commit message: PCB draft
Parts:
- added C1, C11, C12, C4, C5: 220n, NevaDA:C_0603, symbol Device:C
- added C10, C6, C7, C8, C9: 10u, NevaDA:C_1206, symbol Device:C
- added C2, C3: 22p, NevaDA:C_0603, symbol Device:C
- added D1: S3M, NevaDA:DO-214AB_SMC, symbol Device:D
- added Q3: L-7113P3C, NevaDA:LED_3.0mm_pin1-anode, symbol Device:Q_Photo_NPN
- added R1: 1k, NevaDA:R_0603, symbol Device:R
- added R12, R13, R2: 10k, NevaDA:R_0603, symbol Device:R
- added R4, R5, R6, R9: 22, NevaDA:R_1206, symbol Device:R
- added TP1, TP2, TP3, TP4: TestPoint, NevaDA:Screw_M3_9mm, symbol Connector:TestPoint
- added U2: L7805CDT, NevaDA:D-PAK, symbol symbol:LM7805_DPAK
- added Y1: 16 MHz, NevaDA:Crystal_HC-49SMD, symbol Device:Crystal_GND2
- J1: renamed from J?; value Screw_Terminal_01x04 -> X977B06; footprint (none) -> NevaDA:Terminal_X977B06; symbol Connector:Screw_Terminal_01x04 -> Connector:Screw_Terminal_01x06
- R10, R11: renamed from R?; value R -> 22; footprint (none) -> NevaDA:R_1206
- R3, R7, R8: renamed from R?; footprint (none) -> NevaDA:R_0603
- gave numbers to parts that had none: 5
Connections:
- net +12V: now also D1.1 (K), R4.2, R9.1; no longer J1.1 (Pin_1)
- net +5V: now also U1.18 (AV), U1.4 (VCC), U1.6 (VCC), C5.1, C7.1, Q3.1 (C), R2.1, U2.3 (VO)
- net GNDD: now also J1.4 (Pin_4), U1.21 (AGND), U1.3 (GND), U1.5 (GND), C1.2, C10.2, C11.2, C12.2, C2.2, C3.2, C4.2, C5.2, C6.2, C7.2, C8.2, C9.2, R12.2, TP1.1, TP2.1, TP3.1, TP4.1, U2.2 (GND), Y1.2
- net OUT1: now also J1.5 (Pin_5); no longer J1.3 (Pin_3)
- net OUT2: now also J1.6 (Pin_6); no longer J1.4 (Pin_4)
- net PWM1: now also U1.14 (OC1B/PB2); no longer U1.13 (OC1A/PB1)
- net PWM2: now also U1.13 (OC1A/PB1); no longer U1.14 (OC1B/PB2)
- net AREF: now reaches U1.20 (AREF)
- net AREF: now also C4.1
- net OPTIC: now reaches U1.25 (PC2)
- net OPTIC: now also C12.1, R13.1
- net SWITCH_CMOS: now reaches U1.32 (INT0/PD2)
- net SWITCH_CMOS: now also C1.1, R1.1, R2.2
- net XTAL1: now reaches U1.7 (PB6/XTAL1)
- net XTAL1: now also C2.1, Y1.3
- net XTAL2: now reaches U1.8 (PB7/XTAL2)
- net XTAL2: now also C3.1, Y1.1
- net at U3.6 (VCC): now also C10.1, C11.1, C8.1, C9.1, R9.2
- new net: D1.2 (A), J1.3 (Pin_3)
- new net: C6.1, R6.1, U2.1 (VI)
- new net: R4.1, R5.2
- new net: R5.1, R6.2
- new net: Q3.2 (E), R12.1, R13.2
- new net SWITCH: J1.1 (Pin_1), R1.2
- no-connect marks 0 -> 2
Other:
- note removed: "PHOTO + POT\n"
- moved on the sheet: J2, Q1, Q2, R10, R11, R3, R7, R8, U1, U3

Commit message: PCB traced
Parts:
- added C13, C14, C15: 220n, NevaDA:C_0603, symbol Device:C
- added D2: TO-5050BC, NevaDA:LED_RGB_5050-6, symbol symbol:LED_RGB_5050BRG
- added R14, R15: 22, NevaDA:R_1206, symbol Device:R
- added R16, R17, R18: 1k, NevaDA:R_0603, symbol Device:R
- added R19, R20: 10k, NevaDA:R_0603, symbol Device:R
- added SW1, SW2: SW, NevaDA:SW_PUSH_6mm, symbol Switch:SW_Push
- added TP5: TestPoint, NevaDA:1Pin, symbol Connector:TestPoint
- TP1, TP3: footprint NevaDA:Screw_M3_9mm -> NevaDA:Screw_M3_6mm
Connections:
- net +5V: now also R19.1, R20.1, TP5.1
- net GNDD: now also C13.2, C14.2, C15.2, D2.1 (BK), D2.2 (RK), D2.3 (GK), SW1.2, SW2.2
- net OPTIC: now also U1.26 (PC3); no longer U1.25 (PC2)
- net RST: now also C13.1
- net BTN1: now reaches U1.1 (INT1/PD3)
- net BTN1: now also C14.1, R19.2, SW1.1
- net BTN2: now reaches U1.2 (T0/PD4)
- net BTN2: now also C15.1, R20.2, SW2.1
- net LED_1: now reaches U1.23 (PC0)
- net LED_1: now also R16.2
- net LED_2: now reaches U1.24 (PC1)
- net LED_2: now also R17.2
- net at Q1.1 (G), R10.1: now also R14.1
- net at Q2.1 (G), R11.1: now also R15.1
- net at R11.2, U3.5 (Z2): now also R15.2
- net at R10.2, U3.7 (Z1): now also R14.2
- new net: D2.4 (GA), R17.1
- new net: D2.5 (RA), R16.1
- new net: D2.6 (BA), R18.1
- new net LED_3: R18.2, U1.25 (PC2)
Other:
- note removed: "BTN"
- moved on the sheet: C1, C12, Q3, R1, R12, R13, R2, R3

Commit message: Gerbers
Changed lines of the file:
@@
 	1    0    0    -1
 $EndComp
-Text Label 5450 7100 0    50   ~ 0
+Text Label 5450 7100 0    50   ~ 8
 MOSI
-Text Label 4650 7000 2    50   ~ 0
+Text Label 4650 7000 2    50   ~ 8
 MISO
-Text Label 4650 7100 2    50   ~ 0
+Text Label 4650 7100 2    50   ~ 8
 SCK
-Text Label 4650 7200 2    50   ~ 0
+Text Label 4650 7200 2    50   ~ 8
 RST
-Text Label 4100 3850 0    50   ~ 0
+Text Label 4100 3850 0    50   ~ 8
 MISO
-Text Label 4100 3950 0    50   ~ 0
+Text Label 4100 3950 0    50   ~ 8
 SCK
-Text Label 2900 3750 2    50   ~ 0
+Text Label 2900 3750 2    50   ~ 8
 RST
-Text Label 4100 3750 0    50   ~ 0
+Text Label 4100 3750 0    50   ~ 8
 MOSI
-Text Label 2950 7200 2    50   ~ 0
+Text Label 2950 7200 2    50   ~ 8
 RST
 $Comp
@@
 Wire Wire Line
 	3100 7200 3100 7050
-Text Label 4100 3650 0    50   ~ 0
+Text Label 4100 3650 0    50   ~ 8
 PWM1
-Text Label 4100 3550 0    50   ~ 0
+Text Label 4100 3550 0    50   ~ 8
 PWM2
-Text Label 8700 4550 2    50   ~ 0
+Text Label 8700 4550 2    50   ~ 8
 PWM1
-Text Label 8700 4950 2    50   ~ 0
+Text Label 8700 4950 2    50   ~ 8
 PWM2
 $Comp
@@
 	-1   0    0    -1
 $EndComp
-Text Label 2000 1500 0    39   ~ 0
+Text Label 2000 1500 0    39   ~ 7
 OUT1
-Text Label 2000 1600 0    39   ~ 0
+Text Label 2000 1600 0    39   ~ 7
 OUT2
 $Comp
@@
 	0    1    -1   0
 $EndComp
-Text Label 10650 4050 0    39   ~ 0
+Text Label 10650 4050 0    39   ~ 7
 OUT1
-Text Label 10650 4950 0    39   ~ 0
+Text Label 10650 4950 0    39   ~ 7
 OUT2
 $Comp
@@
 Wire Wire Line
 	2000 1400 2200 1400
-Text Label 2000 1100 0    39   ~ 0
+Text Label 2000 1100 0    39   ~ 7
 SWITCH
 Wire Wire Line
@@
 	7400 1650 7400 1800
 Connection ~ 7400 1800
-Text Label 6950 1800 2    39   ~ 0
+Text Label 6950 1800 2    39   ~ 7
 SWITCH
-Text Label 7550 1800 0    39   ~ 0
+Text Label 7550 1800 0    39   ~ 7
 SWITCH_CMOS
 Wire Wire Line
 	7550 1800 7400 1800
-Text Label 4100 5050 0    39   ~ 0
+Text Label 4100 5050 0    39   ~ 7
 SWITCH_CMOS
 NoConn ~ 2900 4250
@@
 	7950 3600 8050 3600
 Connection ~ 7950 3600
-Text Label 8050 3600 0    50   ~ 0
+Text Label 8050 3600 0    50   ~ 8
 OPTIC
-Text Label 4100 4450 0    50   ~ 0
+Text Label 4100 4450 0    50   ~ 8
 OPTIC
 $Comp
@@
 	1    0    0    -1
 $EndComp
-Text Label 2300 4950 0    39   ~ 0
+Text Label 2300 4950 0    39   ~ 7
 XTAL1
-Text Label 2300 5450 0    39   ~ 0
+Text Label 2300 5450 0    39   ~ 7
 XTAL2
-Text Label 2600 4050 0    39   ~ 0
+Text Label 2600 4050 0    39   ~ 7
 AREF
 $Comp
@@
 	9950 5500 9950 5150
 Connection ~ 9950 5150
-Text Label 4100 4150 0    50   ~ 0
+Text Label 4100 4150 0    50   ~ 8
 LED_1
-Text Label 4100 4250 0    50   ~ 0
+Text Label 4100 4250 0    50   ~ 8
 LED_2
-Text Label 4100 4350 0    50   ~ 0
+Text Label 4100 4350 0    50   ~ 8
 LED_3
-Text Label 5400 4400 2    50   ~ 0
+Text Label 5400 4400 2    50   ~ 8
 LED_1
-Text Label 5400 4600 2    50   ~ 0
+Text Label 5400 4600 2    50   ~ 8
 LED_2
-Text Label 5400 4800 2    50   ~ 0
+Text Label 5400 4800 2    50   ~ 8
 LED_3
 $Comp
@@
 	0    -1   -1   0
 $EndComp
-Text Label 5600 5450 2    50   ~ 0
+Text Label 5600 5450 2    50   ~ 8
 BTN1
-Text Label 5600 5850 2    50   ~ 0
+Text Label 5600 5850 2    50   ~ 8
 BTN2
-Text Label 4100 5150 0    50   ~ 0
+Text Label 4100 5150 0    50   ~ 8
 BTN1
-Text Label 4100 5250 0    50   ~ 0
+Text Label 4100 5250 0    50   ~ 8
 BTN2
 $Comp
@@
 	1    0    0    -1
 $EndComp
-Text Label 4000 7200 2    50   ~ 0
+Text Label 4000 7200 2    50   ~ 8
 BTN2
-Text Label 3500 7200 2    50   ~ 0
+Text Label 3500 7200 2    50   ~ 8
 BTN1
 $Comp
